File: 24V Regulator Breakout/24V Regulator Breakout.kicad_pcb (KiCad board)
At the start: 2 copper layers, 61 x 27.9 mm, 9 parts, among them U1 PKE3316ZPI

Commit message: Added Silkscreen
Other:
- board text added: "24V Converter Breakout Mars Rover Design Team Missouri S&T, 2024 Garrett McEntire"
- board text added: "GND"
- board text added: "VIN"
- board text added: "VOUT"
Changed lines of the file:
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@@
   (gr_rect (start 66.04 46.99) (end 127 74.93)
     (stroke (width 0.1) (type default)) (fill none) (layer "Edge.Cuts"))
+  (gr_text "24V Converter Breakout\nMars Rover Design Team\nMissouri S&T, 2024\nGarrett McEntire\n" (at 89.916 74.676 270) (layer "B.SilkS")
+    (effects (font (size 1 1) (thickness 0.15)) (justify left bottom mirror))
+  )
+  (gr_text "VIN\n" (at 76.454 65.024) (layer "F.SilkS")
+    (effects (font (size 1 1) (thickness 0.15)) (justify left bottom))
+  )
+  (gr_text "GND" (at 114.046 58.166) (layer "F.SilkS")
+    (effects (font (size 1 1) (thickness 0.15)) (justify left bottom))
+  )
+  (gr_text "GND" (at 76.454 58.166) (layer "F.SilkS")
+    (effects (font (size 1 1) (thickness 0.15)) (justify left bottom))
+  )
+  (gr_text "VOUT\n" (at 113.284 65.024) (layer "F.SilkS")
+    (effects (font (size 1 1) (thickness 0.15)) (justify left bottom))
+  )
   (segment (start 77.597 62.23) (end 81.788 62.23) (width 0.635) (layer "F.Cu") (net 1))
   (segment (start 81.788 62.23) (end 83.058 63.5) (width 0.635) (layer "F.Cu") (net 1))

Commit message: Fixed Capacitor
Parts:
- C1: value 0.1uF -> 22uF; footprint Capacitor_SMD:C_0603_1608Metric_Pad1.08x0.95mm_HandSolder -> Capacitor_THT:CP_Radial_D5.0mm_P2.00mm
- moved V2 3.81 mm to (127.0, 71.1)
- moved V3 3.81 mm to (127.0, 50.8)
- moved Conn1 3.56 mm to (119.6, 59.7)
- moved C1 1.93 mm to (113.8, 60.3)
- moved C2 0.51 mm to (108.5, 60.7)
Other:
- board size 61 x 27.9 mm -> 64.8 x 27.9 mm
